File: sim_switch/sim_switch.kicad_pcb (KiCad board)
At the start: 2 copper layers, 28 x 43.5 mm, 7 parts, among them U1 SIM800C_Breakout_Board, U2 LM7812_TO220, U3 Mxuteuk_Latching_Mini_Switch, U4 Two_Cables, U5 Two_Cables

Commit message: Sim Switch project improvements
Parts:
- moved H1 0.50 mm to (165.5, 57.0)
- moved H2 0.50 mm to (165.5, 95.0)
Other:
- board size 28 x 43.5 mm -> 28 x 43 mm
- board text added: "CIROTEC AUTOMATION"
Changed lines of the file:
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@@
 			(plot_on_all_layers_selection 0x0000000_00000000)
 			(disableapertmacros no)
-			(usegerberextensions yes)
+			(usegerberextensions no)
 			(usegerberattributes no)
 			(usegerberadvancedattributes no)
@@
 			(psa4output no)
 			(plotreference yes)
-			(plotvalue yes)
+			(plotvalue no)
 			(plotfptext yes)
 			(plotinvisibletext no)
 			(sketchpadsonfab no)
-			(subtractmaskfromsilk no)
+			(subtractmaskfromsilk yes)
 			(outputformat 1)
 			(mirror no)
@@
 	(footprint "MountingHole:MountingHole_2.1mm"
 		(layer "F.Cu")
-		(at 166 57)
+		(at 165.5 57)
 		(descr "Mounting Hole 2.1mm, no annular")
 		(tags "mounting hole 2.1mm no annular")
@@
 			)
 		)
-		(pad "" np_thru_hole circle
+		(pad "" np_thru_hole oval
 			(at 0 0)
-			(size 2.1 2.1)
-			(drill 2.1)
-			(layers "*.Cu" "*.Mask")
+			(size 3.1 2.1)
+			(drill oval 3.1 2.1)
+			(layers "F&B.Cu" "*.Mask")
 		)
 	)
@@
 		(at 153.5 92.5)
 		(property "Reference" "U4"
-			(at -1 -6.5 0)
+			(at -2.5 0 0)
 			(unlocked yes)
 			(layer "F.SilkS")
@@
 		(at 153.5 60 180)
 		(property "Reference" "U5"
-			(at 5 4.5 0)
+			(at 3 -0.5 0)
 			(unlocked yes)
 			(layer "F.SilkS")
@@
 		(at 145 85)
 		(property "Reference" "U1"
-			(at -24 6.5 0)
+			(at -0.5 3 0)
 			(unlocked yes)
 			(layer "F.SilkS")
@@
 				)
 				(justify left bottom)
-			)
-		)
-		(fp_text user "${REFERENCE}"
-			(at -24 9.5 0)
-			(unlocked yes)
-			(layer "F.Fab")
-			(effects
-				(font
-					(size 1 1)
-					(thickness 0.15)
-				)
 			)
 		)
@@
 	(footprint "MountingHole:MountingHole_2.1mm"
 		(layer "F.Cu")
-		(at 166 95)
+		(at 165.5 95)
 		(descr "Mounting Hole 2.1mm, no annular")
 		(tags "mounting hole 2.1mm no annular")
@@
 			)
 		)
-		(pad "" np_thru_hole circle
+		(pad "" np_thru_hole oval
 			(at 0 0)
-			(size 2.1 2.1)
-			(drill 2.1)
-			(layers "*.Cu" "*.Mask")
+			(size 3.1 2.1)
+			(drill oval 3.1 2.1)
+			(layers "F&B.Cu" "*.Mask")
 		)
 	)
 	(gr_rect
 		(start 140 54.5)
-		(end 168 98)
+		(end 168 97.5)
 		(stroke
 			(width 0.05)
@@
 	)
 	(gr_text "INPUT"
-		(at 151 93 0)
+		(at 153 93 0)
 		(layer "F.SilkS")
 		(effects
@@
 		)
 	)
-	(gr_text "OUTPUT"
-		(at 151 61 0)
+	(gr_text "CIROTEC\nAUTOMATION"
+		(at 140.5 58 0)
 		(layer "F.SilkS")
 		(effects
+			(font
+				(size 1 1)
+				(thickness 0.15)
+			)
+			(justify left bottom)
+		)
+	)
+	(gr_text "OUTPUT"
+		(at 152 61 0)
+		(layer "F.SilkS")
+		(effects
